File: kicad/first.sch (KiCad schematic (older format))
At the start: 6 parts, among them J1 Conn_01x05, U1 PIC32MZ2048EFH100, U2 PIC18LF46K22

Commit message: Media migration.
Connections:
- net SPIDOUT is gone; now on net PISPIDOUT: U2.2 (RD4/AN24/P2D/SD02)
Changed lines of the file:
@@
 PGClock
 $Comp
-L GND #PWR01
+L GND #PWR16
 U 1 1 5A48939A
 P 12700 1600
-F 0 "#PWR01" H 12700 1350 50  0001 C CNN
+F 0 "#PWR16" H 12700 1350 50  0001 C CNN
 F 1 "GND" H 12700 1450 50  0000 C CNN
 F 2 "" H 12700 1600 50  0001 C CNN
@@
 $EndComp
 $Comp
-L +3.3V #PWR02
+L +3.3V #PWR17
 U 1 1 5A48944A
 P 12750 700
-F 0 "#PWR02" H 12750 550 50  0001 C CNN
+F 0 "#PWR17" H 12750 550 50  0001 C CNN
 F 1 "+3.3V" H 12750 840 50  0000 C CNN
 F 2 "" H 12750 700 50  0001 C CNN
@@
 NoConn ~ 8900 4500
 $Comp
-L GND #PWR03
+L GND #PWR1
 U 1 1 5A5B002A
 P 600 2800
-F 0 "#PWR03" H 600 2550 50  0001 C CNN
+F 0 "#PWR1" H 600 2550 50  0001 C CNN
 F 1 "GND" H 600 2650 50  0000 C CNN
 F 2 "" H 600 2800 50  0001 C CNN
@@
 $EndComp
 $Comp
-L GND #PWR04
+L GND #PWR2
 U 1 1 5A5B0044
 P 600 5150
-F 0 "#PWR04" H 600 4900 50  0001 C CNN
+F 0 "#PWR2" H 600 4900 50  0001 C CNN
 F 1 "GND" H 600 5000 50  0000 C CNN
 F 2 "" H 600 5150 50  0001 C CNN
@@
 $EndComp
 $Comp
-L GND #PWR05
+L GND #PWR3
 U 1 1 5A5B005E
 P 600 6550
-F 0 "#PWR05" H 600 6300 50  0001 C CNN
+F 0 "#PWR3" H 600 6300 50  0001 C CNN
 F 1 "GND" H 600 6400 50  0000 C CNN
 F 2 "" H 600 6550 50  0001 C CNN
@@
 $EndComp
 $Comp
-L GND #PWR06
+L GND #PWR7
 U 1 1 5A5B00AB
 P 7850 1800
-F 0 "#PWR06" H 7850 1550 50  0001 C CNN
+F 0 "#PWR7" H 7850 1550 50  0001 C CNN
 F 1 "GND" H 7850 1650 50  0000 C CNN
 F 2 "" H 7850 1800 50  0001 C CNN
@@
 $EndComp
 $Comp
-L GND #PWR07
+L GND #PWR9
 U 1 1 5A5B00D1
 P 7850 2800
-F 0 "#PWR07" H 7850 2550 50  0001 C CNN
+F 0 "#PWR9" H 7850 2550 50  0001 C CNN
 F 1 "GND" H 7850 2650 50  0000 C CNN
 F 2 "" H 7850 2800 50  0001 C CNN
@@
 $EndComp
 $Comp
-L GND #PWR08
+L GND #PWR10
 U 1 1 5A5B00EB
 P 7850 4000
-F 0 "#PWR08" H 7850 3750 50  0001 C CNN
+F 0 "#PWR10" H 7850 3750 50  0001 C CNN
 F 1 "GND" H 7850 3850 50  0000 C CNN
 F 2 "" H 7850 4000 50  0001 C CNN
@@
 $EndComp
 $Comp
-L GND #PWR09
+L GND #PWR12
 U 1 1 5A5B0105
 P 7850 5450
-F 0 "#PWR09" H 7850 5200 50  0001 C CNN
+F 0 "#PWR12" H 7850 5200 50  0001 C CNN
 F 1 "GND" H 7850 5300 50  0000 C CNN
 F 2 "" H 7850 5450 50  0001 C CNN
@@
 $EndComp
 $Comp
-L GND #PWR010
+L GND #PWR14
 U 1 1 5A5B011F
 P 7850 6250
-F 0 "#PWR010" H 7850 6000 50  0001 C CNN
+F 0 "#PWR14" H 7850 6000 50  0001 C CNN
 F 1 "GND" H 7850 6100 50  0000 C CNN
 F 2 "" H 7850 6250 50  0001 C CNN
@@
 	7850 3700 8900 3700
 $Comp
-L GND #PWR011
+L GND #PWR19
 U 1 1 5A5B043B
 P 13400 3800
-F 0 "#PWR011" H 13400 3550 50  0001 C CNN
+F 0 "#PWR19" H 13400 3550 50  0001 C CNN
 F 1 "GND" H 13400 3650 50  0000 C CNN
 F 2 "" H 13400 3800 50  0001 C CNN
@@
 	12700 1250 12700 1600
 $Comp
-L +3.3V #PWR012
+L +3.3V #PWR15
 U 1 1 5A5B04FF
 P 7950 3600
-F 0 "#PWR012" H 7950 3450 50  0001 C CNN
+F 0 "#PWR15" H 7950 3450 50  0001 C CNN
 F 1 "+3.3V" H 7950 3740 50  0000 C CNN
 F 2 "" H 7950 3600 50  0001 C CNN
@@
 Connection ~ 7950 3800
 $Comp
-L +3.3V #PWR013
+L +3.3V #PWR18
 U 1 1 5A5B0584
 P 13400 3700
-F 0 "#PWR013" H 13400 3550 50  0001 C CNN
+F 0 "#PWR18" H 13400 3550 50  0001 C CNN
 F 1 "+3.3V" H 13400 3840 50  0000 C CNN
 F 2 "" H 13400 3700 50  0001 C CNN
@@
 	13400 3700 12600 3700
 $Comp
-L +3.3V #PWR014
+L +3.3V #PWR8
 U 1 1 5A5B05CC
 P 7850 2700
-F 0 "#PWR014" H 7850 2550 50  0001 C CNN
+F 0 "#PWR8" H 7850 2550 50  0001 C CNN
 F 1 "+3.3V" H 7850 2840 50  0000 C CNN
 F 2 "" H 7850 2700 50  0001 C CNN
@@
 	6600 2700 7850 2700
 $Comp
-L +3.3V #PWR015
+L +3.3V #PWR11
 U 1 1 5A5B0676
 P 7850 5350
-F 0 "#PWR015" H 7850 5200 50  0001 C CNN
+F 0 "#PWR11" H 7850 5200 50  0001 C CNN
 F 1 "+3.3V" H 7850 5490 50  0000 C CNN
 F 2 "" H 7850 5350 50  0001 C CNN
@@
 	7850 5350 6600 5350
 $Comp
-L +3.3V #PWR016
+L +3.3V #PWR13
 U 1 1 5A5B06BE
 P 7850 6150
-F 0 "#PWR016" H 7850 6000 50  0001 C CNN
+F 0 "#PWR13" H 7850 6000 50  0001 C CNN
 F 1 "+3.3V" H 7850 6290 50  0000 C CNN
 F 2 "" H 7850 6150 50  0001 C CNN
@@
 $EndComp
 $Comp
-L +3.3V #PWR017
+L +3.3V #PWR6
 U 1 1 5A5B078F
 P 700 6450
-F 0 "#PWR017" H 700 6300 50  0001 C CNN
+F 0 "#PWR6" H 700 6300 50  0001 C CNN
 F 1 "+3.3V" H 700 6590 50  0000 C CNN
 F 2 "" H 700 6450 50  0001 C CNN
@@
 $EndComp
 $Comp
-L +3.3V #PWR018
+L +3.3V #PWR5
 U 1 1 5A5B07A9
 P 700 5050
-F 0 "#PWR018" H 700 4900 50  0001 C CNN
+F 0 "#PWR5" H 700 4900 50  0001 C CNN
 F 1 "+3.3V" H 700 5190 50  0000 C CNN
 F 2 "" H 700 5050 50  0001 C CNN
@@
 $EndComp
 $Comp
-L +3.3V #PWR019
+L +3.3V #PWR4
 U 1 1 5A5B07C3
 P 700 2700
-F 0 "#PWR019" H 700 2550 50  0001 C CNN
+F 0 "#PWR4" H 700 2550 50  0001 C CNN
 F 1 "+3.3V" H 700 2840 50  0000 C CNN
 F 2 "" H 700 2700 50  0001 C CNN
@@
 	6600 5250 7200 5250
 Text GLabel 8450 3300 0    51   BiDi ~ 0
-SPIDOUT
+PISPIDOUT
 Text GLabel 8450 3400 0    51   BiDi ~ 0
 RD5
